Commit message: more updates to super Mi experiments

File: husky_description/urdf/accessories/kinect_camera.urdf.xacro (robot description, xacro)
@@ -54,5 +54,5 @@
         <update_rate>20.0</update_rate>
         <camera>
-          <horizontal_fov>${60.0*M_PI/180.0}</horizontal_fov>
+          <horizontal_fov>${70.0*M_PI/180.0}</horizontal_fov>
           <image>
             <format>R8G8B8</format>
@@ -61,6 +61,6 @@
           </image>
           <clip>
-            <near>0.05</near>
-            <far>8.0</far>
+            <near>0.025</near>
+            <far>10.0</far>
           </clip>
         </camera>

File: husky_description/urdf/husky.urdf.xacro (robot description, xacro)
@@ -23,9 +23,9 @@
 <robot name="husky" xmlns:xacro="http://ros.org/wiki/xacro">
   <xacro:arg name="laser_enabled" default="false" />
-  <xacro:arg name="laser_xyz" default="$(optenv HUSKY_LMS1XX_XYZ 0.2206 0.0 0.00635)" />
+  <xacro:arg name="laser_xyz" default="$(optenv HUSKY_LMS1XX_XYZ -0.15 0.0 0.00635)" />
   <xacro:arg name="laser_rpy" default="$(optenv HUSKY_LMS1XX_RPY 0.0 0.0 0.0)" />
   <xacro:arg name="kinect_enabled" default="false" />
-  <xacro:arg name="kinect_xyz" default="$(optenv HUSKY_KINECT_XYZ 0 0 0)" />
-  <xacro:arg name="kinect_rpy" default="$(optenv HUSKY_KINECT_RPY 0 0.18 3.14)" />
+  <xacro:arg name="kinect_xyz" default="$(optenv HUSKY_KINECT_XYZ -0.15 0 0.25)" />
+  <xacro:arg name="kinect_rpy" default="$(optenv HUSKY_KINECT_RPY 0 0.4 0)" />
   <xacro:property name="husky_bumper_extend" value="$(optenv HUSKY_FORWARD_BUMPER_EXTEND 0)" />
   <xacro:arg name="robot_namespace" default="/" />
@@ -36,5 +36,5 @@
   <xacro:include filename="$(find husky_description)/urdf/accessories/kinect_camera.urdf.xacro"/>
   <xacro:include filename="$(find husky_description)/urdf/accessories/sick_lms1xx_mount.urdf.xacro"/>
-  <xacro:include filename="$(find husky_description)/urdf/accessories/sensor_arch.urdf.xacro"/>
+  <!-- <xacro:include filename="$(find husky_description)/urdf/accessories/sensor_arch.urdf.xacro"/> -->
   <xacro:property name="M_PI" value="3.14159"/>
   <!-- Base Size -->
@@ -124,10 +124,10 @@
   </xacro:if>
   <xacro:if value="$(arg kinect_enabled)">
-    <xacro:sensor_arch prefix="" parent="top_plate_link">
+    <!-- <xacro:sensor_arch prefix="" parent="top_plate_link">
       <origin xyz="-0.35 0 0.51" rpy="0 0 -3.14"/>
-    </xacro:sensor_arch>
+    </xacro:sensor_arch> -->
     <joint name="kinect_frame_joint" type="fixed">
       <origin xyz="$(arg kinect_xyz)" rpy="$(arg kinect_rpy)" />
-      <parent link="sensor_arch_mount_link"/>
+      <parent link="top_plate_link"/>
       <child link="camera_link"/>
     </joint>
